Commit message: fixed xacro:include tags and added inertial tags

File: cfg/s-model_articulated.urdf (robot description, URDF)
Before this commit: robot s-model_articulated, 13 links, 12 joints
Links:
- link finger_1_link_0: mass None -> 0.05
- link finger_1_link_1: mass None -> 0.15
- link finger_1_link_2: mass None -> 0.15
- link finger_1_link_3: mass None -> 0.05
- link finger_2_link_0: mass None -> 0.05
- link finger_2_link_1: mass None -> 0.15
- link finger_2_link_2: mass None -> 0.15
- link finger_2_link_3: mass None -> 0.05
- link finger_middle_link_0: mass None -> 0.05
- link finger_middle_link_1: mass None -> 0.15
- link finger_middle_link_2: mass None -> 0.15
- link finger_middle_link_3: mass None -> 0.05

File: cfg/s-model_articulated.xacro (robot description, xacro)
@@ -5,5 +5,5 @@
 -->
 <robot name="s-model_articulated" xmlns:xacro="http://ros.org/wiki/xacro">
-	<include filename="$(find robotiq_s_model_visualization)/cfg/s-model_articulated_macro.xacro" />
+	<xacro:include filename="$(find robotiq_s_model_visualization)/cfg/s-model_articulated_macro.xacro" />
 	<xacro:s-model_articulated prefix=""/>
 <!--

File: cfg/s-model_articulated_macro.xacro (robot description, xacro)
@@ -6,5 +6,5 @@
 -->
 <robot xmlns:xacro="http://ros.org/wiki/xacro">
-	<include filename="$(find robotiq_s_model_visualization)/cfg/s-model_finger_articulated_macro.xacro" />
+	<xacro:include filename="$(find robotiq_s_model_visualization)/cfg/s-model_finger_articulated_macro.xacro" />
 	<xacro:macro name="s-model_articulated" params="prefix">
 	<xacro:s-model_finger_articulated prefix="${prefix}finger_1_"/>
@@ -30,4 +30,9 @@
 			</collision>
 		</link>
+        <inertial>
+            <origin xyz="0 0 0" rpy="0 0 0"/>
+            <mass value="1.3"/>
+            <inertia ixx="0.006012" ixy="0.000079" ixz="-0.00024" iyy="0.012892" iyz="0" izz="0.002435" />
+        </inertial>
 		<!-- end of link list -->
 		<!-- joint list -->

File: cfg/s-model_finger_articulated_macro.xacro (robot description, xacro)
@@ -27,4 +27,9 @@
 				</material>
 			</collision>
+            <inertial>
+                <origin xyz="0 0 0" rpy="0 0 0"/>
+                <mass value="0.05"/>
+                <inertia ixx="0.01" ixy="-0.00002" ixz="0.00001" iyy="0.0008" iyz="0" izz="0.001" />
+            </inertial>
 		</link>
 		<link name="${prefix}link_1">
@@ -43,4 +48,9 @@
 				<material name="yellow"/>
 			</collision>
+            <inertial>
+                <origin xyz="0 0 0" rpy="0 0 0"/>
+                <mass value="0.15"/>
+                <inertia ixx="0.001859" ixy="-0.000376" ixz="0.000028" iyy="0.012756" iyz="0" izz="0.0024" />
+            </inertial>
 		</link>
 		<link name="${prefix}link_2">
@@ -64,4 +74,9 @@
 				<material name="yellow"/>
 			</collision>
+            <inertial>
+                <origin xyz="0 0 0" rpy="0 0 0"/>
+                <mass value="0.15"/>
+                <inertia ixx="0.001859" ixy="-0.000376" ixz="0.000028" iyy="0.012756" iyz="0" izz="0.0024" />
+            </inertial>
 		</link>
 		<link name="${prefix}link_3">
@@ -80,4 +95,9 @@
 				<material name="yellow"/>
 			</collision>
+            <inertial>
+                <origin xyz="0 0 0" rpy="0 0 0"/>
+                <mass value="0.05"/>
+                <inertia ixx="0.001239" ixy="-0.000251" ixz="0.000019" iyy="0.00085" iyz="0" izz="0.001632" />
+            </inertial>
 		</link>
 		<!-- end of link list -->
